File: trunk/Hardware/Eagle/Touch_Panel/Module Touch Panel/Generic Electronics Board (PCB B)/Generic Electronics Board (PCB B).brd (EAGLE design)
At the start: 45.6 x 36.9 mm, 54 parts, among them IC1 ST3485, IC3 DS18B20, U1 XMEGA-A4TQFP, U2 SPX1117M3-L-3-3, X1 RJ45-8L-B, X6 RJ45-8L-B

Commit message: Minor changes
Parts:
- C4: value 4n7 -> 4n7 (22n)
Routing:
- net GND_RS485: track 36.0 -> 38.6 mm
- net Y1: track 15.8 -> 16.4 mm
Changed lines of the file:
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@@
 <setting verticaltext="up"/>
 </settings>
-<grid distance="0.05" unitdist="inch" unit="mm" style="lines" multiple="1" display="no" altdistance="0.1" altunitdist="mm" altunit="mm"/>
+<grid distance="0.05" unitdist="inch" unit="mil" style="lines" multiple="1" display="no" altdistance="0.1" altunitdist="mm" altunit="mm"/>
 <layers>
 <layer number="1" name="Top" color="4" fill="1" visible="yes" active="yes"/>
@@
 <layer number="17" name="Pads" color="2" fill="1" visible="yes" active="yes"/>
 <layer number="18" name="Vias" color="2" fill="1" visible="yes" active="yes"/>
-<layer number="19" name="Unrouted" color="6" fill="1" visible="no" active="yes"/>
+<layer number="19" name="Unrouted" color="6" fill="1" visible="yes" active="yes"/>
 <layer number="20" name="Dimension" color="15" fill="1" visible="yes" active="yes"/>
-<layer number="21" name="tPlace" color="7" fill="1" visible="no" active="yes"/>
-<layer number="22" name="bPlace" color="7" fill="1" visible="no" active="yes"/>
-<layer number="23" name="tOrigins" color="15" fill="1" visible="no" active="yes"/>
-<layer number="24" name="bOrigins" color="15" fill="1" visible="no" active="yes"/>
-<layer number="25" name="tNames" color="7" fill="1" visible="no" active="yes"/>
-<layer number="26" name="bNames" color="7" fill="1" visible="no" active="yes"/>
+<layer number="21" name="tPlace" color="7" fill="1" visible="yes" active="yes"/>
+<layer number="22" name="bPlace" color="7" fill="1" visible="yes" active="yes"/>
+<layer number="23" name="tOrigins" color="15" fill="1" visible="yes" active="yes"/>
+<layer number="24" name="bOrigins" color="15" fill="1" visible="yes" active="yes"/>
+<layer number="25" name="tNames" color="7" fill="1" visible="yes" active="yes"/>
+<layer number="26" name="bNames" color="7" fill="1" visible="yes" active="yes"/>
 <layer number="27" name="tValues" color="7" fill="1" visible="no" active="yes"/>
 <layer number="28" name="bValues" color="7" fill="1" visible="no" active="yes"/>
@@
 <layer number="45" name="Holes" color="7" fill="1" visible="no" active="yes"/>
 <layer number="46" name="Milling" color="3" fill="1" visible="no" active="yes"/>
-<layer number="47" name="Measures" color="7" fill="1" visible="no" active="yes"/>
-<layer number="48" name="Document" color="7" fill="1" visible="no" active="yes"/>
+<layer number="47" name="Measures" color="7" fill="1" visible="yes" active="yes"/>
+<layer number="48" name="Document" color="7" fill="1" visible="yes" active="yes"/>
 <layer number="49" name="Reference" color="7" fill="1" visible="yes" active="yes"/>
 <layer number="50" name="dxf" color="7" fill="1" visible="no" active="no"/>
-<layer number="51" name="tDocu" color="7" fill="1" visible="no" active="yes"/>
-<layer number="52" name="bDocu" color="7" fill="1" visible="no" active="yes"/>
+<layer number="51" name="tDocu" color="7" fill="1" visible="yes" active="yes"/>
+<layer number="52" name="bDocu" color="7" fill="1" visible="yes" active="yes"/>
 <layer number="91" name="Nets" color="2" fill="1" visible="no" active="no"/>
 <layer number="92" name="Busses" color="1" fill="1" visible="no" active="no"/>
@@
 <layer number="103" name="tMap" color="7" fill="1" visible="no" active="yes"/>
 <layer number="104" name="Name" color="7" fill="1" visible="no" active="yes"/>
-<layer number="105" name="tPlate" color="7" fill="1" visible="no" active="yes"/>
-<layer number="106" name="bPlate" color="7" fill="1" visible="no" active="yes"/>
+<layer number="105" name="tPlate" color="7" fill="1" visible="yes" active="yes"/>
+<layer number="106" name="bPlate" color="7" fill="1" visible="yes" active="yes"/>
 <layer number="107" name="Crop" color="7" fill="1" visible="no" active="yes"/>
 <layer number="116" name="Patch_BOT" color="7" fill="1" visible="no" active="yes"/>
@@
 <element name="R14" library="rcl" package="R0603" value="1k" x="67.24" y="33.05" rot="MR270"/>
 <element name="C1" library="rcl" package="C0603" value="4n7" x="78.11" y="45.55" rot="MR270"/>
-<element name="C4" library="rcl" package="C0603" value="4n7" x="80.86" y="45.55" rot="MR270"/>
+<element name="C4" library="rcl" package="C0603" value="4n7 (22n)" x="80.86" y="45.55" rot="MR270"/>
 <element name="C7" library="rcl" package="C0603" value="4n7" x="79.44" y="45.52" rot="MR270"/>
 <element name="R15" library="rcl" package="R0603" value="470k" x="80.46" y="51.12" rot="R270"/>
@@
 <contactref element="IC3" pad="1"/>
 <contactref element="IC3" pad="1"/>
-<wire x1="55.65" y1="40.47" x2="56.505" y2="39.615" width="0.254" layer="1"/>
+<wire x1="55.65" y1="40.47" x2="56.505" y2="39.615" width="0.6096" layer="1"/>
 <wire x1="56.505" y1="39.615" x2="56.505" y2="39.405" width="0.254" layer="1"/>
 <contactref element="R24" pad="1"/>
@@
 <wire x1="79.4" y1="40.9" x2="79.4" y2="41" width="0.254" layer="1"/>
 <wire x1="79.4" y1="41" x2="79.4" y2="40.9" width="0.254" layer="1"/>
-<wire x1="79.39" y1="32.69" x2="77.3" y2="30.6" width="0.254" layer="1"/>
-<wire x1="77.3" y1="30.6" x2="75.06" y2="30.6" width="0.254" layer="1"/>
-<wire x1="75.06" y1="30.6" x2="73.82" y2="29.36" width="0.254" layer="1"/>
+<wire x1="79.29" y1="31.52" x2="78.17" y2="30.4" width="0.254" layer="1"/>
+<wire x1="78.17" y1="30.4" x2="74.96" y2="30.4" width="0.254" layer="1"/>
+<wire x1="74.96" y1="30.4" x2="73.82" y2="29.36" width="0.254" layer="1"/>
 <wire x1="79.4" y1="40.9" x2="79.39" y2="40.9" width="0.254" layer="1"/>
 <wire x1="79.4" y1="40.9" x2="79.4" y2="40.1" width="0.254" layer="1"/>
 <wire x1="79.4" y1="40.1" x2="79.9" y2="39.6" width="0.254" layer="1"/>
-<wire x1="79.9" y1="39.6" x2="79.9" y2="33.2" width="0.254" layer="1"/>
-<wire x1="79.9" y1="33.2" x2="79.39" y2="32.69" width="0.254" layer="1"/>
+<wire x1="79.9" y1="39.6" x2="79.9" y2="32.13" width="0.254" layer="1"/>
+<wire x1="79.9" y1="32.13" x2="79.29" y2="31.52" width="0.254" layer="1"/>
 </signal>
 <signal name="Y2">
@@
 <contactref element="R10" pad="1"/>
 <contactref element="X1" pad="8"/>
-<wire x1="56.65" y1="30.1" x2="57.25" y2="29.45" width="0.3048" layer="1"/>
-<wire x1="57.25" y1="29.45" x2="58.9" y2="27.8" width="0.3048" layer="1"/>
-<wire x1="58.9" y1="27.8" x2="58.9" y2="24.025" width="0.3048" layer="1"/>
-<wire x1="58.9" y1="24.025" x2="58.925" y2="24" width="0.3048" layer="1"/>
-<wire x1="58.925" y1="24" x2="76.6" y2="24" width="0.3048" layer="1"/>
-<wire x1="76.6" y1="24" x2="77.8" y2="25.2" width="0.3048" layer="1"/>
-<wire x1="77.8" y1="25.2" x2="85.665" y2="25.2" width="0.3048" layer="1"/>
-<wire x1="85.665" y1="25.2" x2="86.865" y2="24" width="0.3048" layer="1"/>
+<wire x1="56.65" y1="30.1" x2="58.7" y2="30.1" width="0.8128" layer="1"/>
+<wire x1="58.7" y1="30.1" x2="59.7" y2="29.1" width="0.8128" layer="1"/>
+<wire x1="59.7" y1="29.1" x2="59.7" y2="24.5" width="0.8128" layer="1"/>
+<wire x1="59.7" y1="24.5" x2="59.1" y2="23.9" width="0.8128" layer="1"/>
+<wire x1="59.1" y1="23.9" x2="59.025" y2="23.9" width="0.254" layer="1"/>
+<wire x1="59.025" y1="23.9" x2="58.925" y2="24" width="0.254" layer="1"/>
+<wire x1="86.865" y1="24" x2="86.865" y2="23.465" width="0.8128" layer="16"/>
+<wire x1="86.865" y1="23.465" x2="85.6" y2="22.4" width="0.8128" layer="16"/>
+<wire x1="85.6" y1="22.4" x2="60.625" y2="22.4" width="0.8128" layer="16"/>
+<wire x1="60.625" y1="22.4" x2="58.925" y2="24" width="0.8128" layer="16"/>
 </signal>
 <signal name="BUS_PWR">
@@
 <contactref element="R14" pad="2"/>
 <wire x1="67.24" y1="32.2" x2="63" y2="32.2" width="0.254" layer="16"/>
-<wire x1="63" y1="32.2" x2="62.1" y2="32.2" width="0.254" layer="16"/>
-<wire x1="62.1" y1="32.2" x2="61.4" y2="31.5" width="0.254" layer="16"/>
-<wire x1="61.4" y1="31.5" x2="61.4" y2="27.6" width="0.254" layer="16"/>
+<wire x1="63" y1="32.2" x2="62.8" y2="32.2" width="0.254" layer="16"/>
+<wire x1="62.8" y1="32.2" x2="61.4" y2="30.8" width="0.254" layer="16"/>
+<wire x1="61.4" y1="30.8" x2="61.4" y2="27.6" width="0.254" layer="16"/>
 <wire x1="61.4" y1="27.6" x2="62.1" y2="26.9" width="0.254" layer="16"/>
 <wire x1="62.1" y1="26.9" x2="63.24" y2="26.9" width="0.254" layer="16"/>

Commit message: PDI signals renamed.
Connections:
- net N$3 renamed PC2
- net N$7 renamed PDI_DATA
- net N$8 renamed PDI_CLK
- net N$9 renamed PC3
Changed lines of the file:
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@@
 <?xml version="1.0" encoding="utf-8"?>
 <!DOCTYPE eagle SYSTEM "eagle.dtd">
-<eagle version="6.1">
+<eagle version="6.4">
 <drawing>
 <settings>
@@
 </class>
 </classes>
-<designrules>
+<designrules name="default">
 <description language="de">&lt;b&gt;EAGLE Design Rules&lt;/b&gt;
 &lt;p&gt;
@@
 <wire x1="65.39" y1="36.1" x2="65.38" y2="36.11" width="0.254" layer="16"/>
 </signal>
-<signal name="N$7">
+<signal name="PDI_DATA">
 <contactref element="U1" pad="34"/>
 <contactref element="JP1" pad="2"/>
@@
 <wire x1="64.57" y1="47.7" x2="64.58" y2="47.71" width="0.254" layer="16"/>
 </signal>
-<signal name="N$8">
+<signal name="PDI_CLK">
 <contactref element="U1" pad="35"/>
 <contactref element="JP1" pad="4"/>
@@
 <wire x1="74.99" y1="37.3" x2="74.38" y2="37.91" width="0.254" layer="16"/>
 </signal>
-<signal name="N$3">
+<signal name="PC2">
 <contactref element="R3" pad="1"/>
 <contactref element="U1" pad="12"/>
@@
 <wire x1="72.99" y1="35.7" x2="72.58" y2="36.11" width="0.254" layer="16"/>
 </signal>
-<signal name="N$9">
+<signal name="PC3">
 <contactref element="R4" pad="1"/>
 <contactref element="U1" pad="13"/>
