File: trunk/Hardware/Eagle/Actor_6_Channel_16A/Actor_6_Channel.brd (EAGLE design)
At the start: 103 x 87.7 mm, 52 parts, among them IC1 ULN2803A, IC2 ST3485, IC3 7824TV, U1 XMEGA-32D4TQFP, U2 SPX1117M3-L-3-3, X6 RJ45-8L-B, X7 RJ45-8L-B

Commit message: Actor 6CH for review
Parts:
- removed C13, C5: 100n, rcl:C0603K
- removed C2: 100n, rcl:C0603
- removed C7: 10uF/50V, rcl:E2,5-5
- removed CH1, CH2, CH3, CH4, CH5, CH6: G2RA, relay:G2RA
- removed D5: (no value), diode:DO214AA
- removed R25: 100k, rcl:R0603
- removed R32: 10k, rcl:R0603
- added K1, K2, K3, K4, K5, K6: RMB841, relay:RT2N/O
- added R10, R11, R12, R14, R18, R19, R20, R3, R9: 100R, rcl:R0603
- added R4, R5: 10R, rcl:R0603
- added R6: 750R, rcl:M1206
- added R8: 750R, rcl:R0603
- IC1: value ULN2803A -> ST3485; device uln-udn:SO18W -> 751xx:D_R-PDSO-G8
- IC2: value ST3485 -> ULN2003AD; device 751xx:D_R-PDSO-G8 -> uln-udn:SO16
- IC3: value 7824TV -> ULN2003AD; device linear:TO220V -> uln-udn:SO16
- JP1: value (none) -> terminator; device pinhead:2X08 -> jumper:JP1
- R13: value 750R -> 100R
- R15: value 750R -> 100R; device rcl:M1206 -> rcl:R0603
- R16, R17: value 10R -> 100R
- R2: value 100R -> 100k
- moved R16 360.7 mm to (-17.1, -299.7), turned to 0 degrees
- moved R17 358.6 mm to (-17.1, -304.8), turned to 0 degrees
- moved R15 354.0 mm to (-17.1, -294.6), turned to 0 degrees
- moved R13 341.5 mm to (-17.1, -284.5), turned to 0 degrees
- moved JP1 307.9 mm to (-22.9, -319.4)
- moved IC2 128.1 mm to (11.4, 37.5), turned to 0 degrees
- moved IC3 111.2 mm to (-11.4, -174.0)
- moved IC1 107.9 mm to (139.1, 26.0), turned to 90 degrees
- moved R2 30.5 mm to (1.91, -36.2)
- renumbered JP8 to JP2, R24 to R1
Connections:
- removed net CH1+: CH1.S, X1.2
- removed net CH2+: CH2.S, X2.1
- removed net N$31: JP1.2, U1.10
- removed net PA0: IC1.1, U1.40
- removed net PA1: IC1.2, U1.41
- removed net PA2: IC1.3, U1.42
- removed net PA3: IC1.6, U1.43
- removed net PA4: IC1.7, U1.44
- removed net PA5: IC1.8, U1.1
- new net K1_0: IC2.16, K1.A2, R9.1
- new net K1_1: IC2.15, K1.A1, R10.1
- new net K2_0: IC2.14, K2.A2, R11.1
- new net K2_1: IC2.13, K2.A1, R12.1
- new net K3_0: IC2.12, K3.A2, R13.1
- new net K3_1: IC2.11, K3.A1, R14.1
- new net K4_0: IC3.16, K4.A2, R15.1
- new net K4_1: IC3.15, K4.A1, R16.1
- new net K5_0: IC3.14, K5.A2, R17.1
- new net K5_1: IC3.13, K5.A1, R18.1
- new net K6_0: IC3.12, K6.A2, R19.1
- new net K6_1: IC3.11, K6.A1, R20.1
- new net N$34: IC2.6, U1.2
- net +24V: now also L1.2, R10.2, R11.2, R12.2, R13.2, R14.2, R15.2, R16.2, R17.2, R18.2, R19.2, R20.2, R9.2; no longer C5.1, CH1.1, CH2.1, CH3.1, CH4.1, CH5.1, CH6.1, D5.A, IC1.10, IC3.3
- net +3V3: now also IC1.8, R8.2; no longer IC2.8, R13.2, R32.2
- net A: now also R5.1; no longer R16.1
- net B: now also R4.1; no longer R17.1
- net GND: now also IC1.5, IC2.8, IC3.8, R3.2, R6.1; no longer C13.2, C2.2, C5.2, C7.-, IC1.9, IC2.5, IC3.2, JP1.15, R15.1, R2.2
- net GND_RS485: now also R3.1; no longer R2.1
- net N$1: now also K1.11, K1.21; no longer CH1.P
- net N$10: now also K5.14, K5.24, X4.1; no longer CH6.2, IC1.11, JP1.13
- net N$11: now also K6.11, K6.21, X4.2; no longer CH5.2, IC1.12, JP1.11
- net N$12: now also K6.14, K6.24, X4.3; no longer CH4.2, IC1.13, JP1.9
- net N$13: now also IC2.1, U1.41; no longer CH5.P, X3.3
- net N$16: now also IC1.7, R4.2, R6.2; no longer IC2.7, R15.2, R17.2
- net N$18: now also IC2.2, U1.42; no longer CH4.P, X3.1
- net N$19: now also IC2.3, U1.43; no longer CH6.P, X4.2
- net N$2: now also K1.14, K1.24, X1.2; no longer CH3.S, X2.3
- net N$20: now also IC2.4, U1.44; no longer CH6.S, X4.3
- net N$21: now also IC3.1, U1.3; no longer JP1.16, U1.17
- net N$22: now also IC3.2, U1.4; no longer JP1.14, U1.16
- net N$23: now also IC3.3, U1.5; no longer JP1.12, U1.15
- net N$24: now also IC1.2, IC1.3; no longer IC2.2, IC2.3
- net N$25: now also IC1.4; no longer IC2.4
- net N$26: now also IC1.1; no longer IC2.1
- net N$27: now also IC3.4, U1.6; no longer JP1.10, U1.14
- net N$28: now also JP1.2; no longer JP1.8
- net N$29: now also JP1.1; no longer JP1.6
- net N$3: now also K2.14, K2.24, X2.1; no longer CH2.P, X1.3
- net N$30: now also IC3.5, U1.7; no longer JP1.4, U1.11
- net N$32: now also IC2.5, U1.1; no longer C13.1, C7.+, D5.C, IC3.1, L1.2
- net N$4: now also K2.11, K2.21, X1.3; no longer CH4.S, X3.2
- net N$5: now also K3.11, K3.21; no longer CH3.P
- net N$6: now also K3.14, K3.24, X2.3; no longer CH5.S, X4.1
- net N$7: now also K4.11, K4.21, X3.1; no longer CH1.2, IC1.18, JP1.3
- net N$8: now also K4.14, K4.24, X3.2; no longer CH2.2, IC1.17, JP1.5
- net N$9: now also K5.11, K5.21, X3.3; no longer CH3.2, IC1.16, JP1.7
- net PROG: no longer C2.1, R32.1
- net RS485_A1: now also IC1.6, R5.2, R8.1; no longer IC2.6, R13.1, R16.2
- net VCC: now also IC2.9, IC3.9; no longer C4.1, D3.C, D4.A, JP1.1
- net VCC_MAG: now also C4.1, D3.C, D4.A, R2.2; no longer R25.2
- net VCC_MAG_METER: now also R2.1, U1.40; no longer R25.1, U1.7

Commit message: Actor_6_Channel.brd FV
Parts:
- added JP4: (no value), pinhead:2X04
- added R21, R22: 0R, rcl:R0603
- C3: device rcl:C0603 -> rcl:C0603K
- moved R20 381.8 mm to (98.2, 43.9), turned to 180 degrees
- moved R19 375.2 mm to (92.3, 43.9)
- moved R18 367.2 mm to (81.0, 43.9), turned to 180 degrees
- moved R17 360.8 mm to (75.2, 43.9)
- moved R16 353.1 mm to (63.9, 43.9), turned to 180 degrees
- moved R15 346.8 mm to (58.0, 43.9)
- moved R14 339.6 mm to (46.7, 43.9), turned to 180 degrees
- moved JP1 337.6 mm to (35.8, 13.1), turned to 180 degrees
- moved R13 333.5 mm to (40.9, 43.9)
- moved R12 326.7 mm to (29.6, 43.9), turned to 180 degrees
- moved R11 320.9 mm to (23.7, 43.9)
- moved R10 314.6 mm to (12.4, 43.9), turned to 180 degrees
- moved R9 309.0 mm to (6.60, 43.9)
- moved IC3 214.2 mm to (36.4, 34.8)
- moved L2 159.7 mm to (42.5, 30.0), turned to 90 degrees
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Connections:
- net N$24 renamed DE_/RE
- net N$25 renamed TXD
- net N$26 renamed RXD
- net VCC_MAG renamed VCC_BUS
- net VCC_MAG_METER renamed VCC_BUS_METER
- removed net GND_RS485: R3.1, X6.2, X6.6, X6.8, X7.2, X7.6, X7.8
- removed net N$13: IC2.1, U1.41
- removed net N$18: IC2.2, U1.42
- removed net N$19: IC2.3, U1.43
- removed net N$20: IC2.4, U1.44
- removed net N$21: IC3.1, U1.3
- removed net N$22: IC3.2, U1.4
- removed net N$23: IC3.3, U1.5
- removed net N$27: IC3.4, U1.6
- removed net N$30: IC3.5, U1.7
- removed net N$32: IC2.5, U1.1
- removed net N$33: JP3.3, U1.35
- removed net N$34: IC2.6, U1.2
- removed net VCC: IC2.9, IC3.9
- new net /LA: JP4.1, U1.24
- new net CLK: JP4.3, U1.27
- new net INT: JP4.6, U1.32
- new net MOSI: JP4.2, U1.25
- new net N$11: JP3.3, U1.34
- new net N$36: C1.2, D1.A, D2.A, IC1.5, R21.2, R3.2, R6.1
- new net N$37: R22.2, R3.1, X6.2, X6.6, X6.8, X7.2, X7.6, X7.8
- new net PA1: IC3.6, U1.41
- new net PA2: IC3.5, U1.42
- new net PA3: IC3.4, U1.43
- new net PA4: IC3.3, U1.44
- new net PA5: IC3.2, U1.1
- new net PA6: IC3.1, U1.2
- new net PA7: IC2.6, U1.3
- new net PB0: IC2.5, U1.4
- new net PB1: IC2.4, U1.5
- new net PB2: IC2.3, U1.6
- new net PB3: IC2.2, U1.7
- new net PC0: IC2.1, U1.10
- new net SCL: JP4.5, U1.29
- new net SDA: JP4.4, U1.28
- net +24V: now also IC2.9, IC3.9
- net +3V3: now also JP4.7
- net GND: now also JP3.1, JP4.8, R21.1, R22.1; no longer C1.2, D1.A, D2.A, IC1.5, JP3.4, R3.2, R6.1
- net K1_1: now also IC3.16; no longer IC2.15
- net K2_0: now also IC2.15; no longer IC2.14
- net K2_1: now also IC3.15; no longer IC2.13
- net K3_0: now also IC2.14; no longer IC2.12
- net K3_1: now also IC3.14; no longer IC2.11
- net K4_0: now also IC2.13; no longer IC3.16
- net K4_1: now also IC3.13; no longer IC3.15
- net K5_0: now also IC2.12; no longer IC3.14
- net K5_1: now also IC3.12; no longer IC3.13
- net K6_0: now also IC2.11; no longer IC3.12
- net N$14: now also JP3.4, U1.35; no longer JP3.1, U1.34
- net PROG: now also U1.14
Routing:
- net +24V: track 0.00 -> 325.9 mm
- net GND: track 0.00 -> 222.0 mm, vias 0 -> 2
- net +3V3: track 0.00 -> 140.5 mm, vias 0 -> 1
- net K6_0: track 0.00 -> 88.3 mm
- net K5_0: track 0.00 -> 75.3 mm
- net K6_1: track 0.00 -> 69.6 mm, vias 0 -> 1
- net N$2: track 0.00 -> 64.7 mm
- net VCC_BUS: track 0.00 -> 63.3 mm
- net K4_0: track 0.00 -> 60.6 mm
- net K5_1: track 0.00 -> 54.3 mm, vias 0 -> 1
- net N$5: track 0.00 -> 53.1 mm
- net N$37: track 0.00 -> 52.0 mm
- net A: track 0.00 -> 46.8 mm
- net PROG: track 0.00 -> 46.7 mm, vias 0 -> 1
- net K3_0: track 0.00 -> 46.0 mm
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- added copper zone on layer 1, net GND
- added copper zone on layer 16, net GND
Other:
- board text added: "Actor 6CH ver. 1.00_20.07.13"
