File: trunk/Hardware/Eagle/Actor_6_Channel_16A/Actor_6_Channel.sch (EAGLE design)
At the start: 52 parts, among them IC1 ULN2803A, IC2 ST3485, IC3 7824TV, U1 XMEGA-32D4TQFP, U2 SPX1117M3-L-3-3, X1 MKDS_5/3-7,5, X2 MKDS_5/3-7,5, X3 MKDS_5/3-7,5, X4 MKDS_5/3-7,5, X6 RJ45-8L-B, X7 RJ45-8L-B

Commit message: Actor 6CH for review
Parts:
- removed C13, C5: 100n, rcl:C-EUC0603K
- removed C2: 100n, rcl:C-EUC0603
- removed C7: 10uF/50V, rcl:CPOL-EUE2.5-5
- removed CH1, CH2, CH3, CH4, CH5, CH6: G2RA, relay:G2RA
- removed D5: (no value), diode:DIODE-DO214AA
- removed R24: 3k65, rcl:R-EU_R0603
- removed R25: 100k, rcl:R-EU_R0603
- removed R32: 10k, rcl:R-EU_R0603
- added K1, K2, K3, K4, K5, K6: RMB841, relay:RT444730
- added R1: 3k65, rcl:R-EU_R0603
- added R10, R11, R12, R14, R18, R19, R20, R3, R9: 100R, rcl:R-EU_R0603
- added R4, R5: 10R, rcl:R-EU_R0603
- added R6: 750R, rcl:R-EU_M1206
- added R8: 750R, rcl:R-EU_R0603
- IC1: value ULN2803A -> ST3485; device uln-udn:ULN2803ASMD_SO18 -> 751xx:75176AD
- IC2: value ST3485 -> ULN2003AD; device 751xx:75176AD -> uln-udn:ULN2003AD
- IC3: value 7824TV -> ULN2003AD; device linear:7824TV -> uln-udn:ULN2003AD
- JP1: value (none) -> terminator; device pinhead:PINHD-2X8 -> jumper:JP1Q
- R13: value 750R -> 100R
- R15: value 750R -> 100R; device rcl:R-EU_M1206 -> rcl:R-EU_R0603
- R16, R17: value 10R -> 100R
- R2: value 100R -> 100k
- renumbered JP8 to JP2
Connections:
- removed net CH1+: CH12.S, X1-2.KL
- removed net CH2+: CH22.S, X2-1.KL
- removed net N$31: JP1.2, U1.PC0(OC0A/SDA)
- removed net PA0: IC1.I1, U1.PA0(ADC0/AREF)
- removed net PA1: IC1.I2, U1.PA1(ADC1)
- removed net PA2: IC1.I3, U1.PA2(ADC2)
- removed net PA3: IC1.I6, U1.PA3(ADC3)
- removed net PA4: IC1.I7, U1.PA4(ADC4)
- removed net PA5: IC1.I8, U1.PA5(ADC5)
- new net K1_0: IC2.O1, K11.1, R9.1
- new net K1_1: IC2.O2, K11.2, R10.1
- new net K2_0: IC2.O3, K21.1, R11.1
- new net K2_1: IC2.O4, K21.2, R12.1
- new net K3_0: IC2.O5, K31.1, R13.1
- new net K3_1: IC2.O6, K31.2, R14.1
- new net K4_0: IC3.O1, K41.1, R15.1
- new net K4_1: IC3.O2, K41.2, R16.1
- new net K5_0: IC3.O3, K51.1, R17.1
- new net K5_1: IC3.O4, K51.2, R18.1
- new net K6_0: IC3.O5, K61.1, R19.1
- new net K6_1: IC3.O6, K61.2, R20.1
- new net N$34: IC2.I6, U1.PA6(ADC6)
- net +24V: now also L1.2, R10.2, R11.2, R12.2, R13.2, R14.2, R15.2, R16.2, R17.2, R18.2, R19.2, R20.2, R9.2; no longer C5.1, CH11.1, CH21.1, CH31.1, CH41.1, CH51.1, CH61.1, D5.A, IC1.CD+, IC3.VO
- net +3V3: now also IC1.VCC, R8.2; no longer IC2.VCC, R13.2, R32.2
- net A: now also R5.1; no longer R16.1
- net B: now also R4.1; no longer R17.1
- net GND: now also R1.1, R3.2, R6.1; no longer C13.2, C2.2, C5.2, C7.-, JP1.15, R15.1, R2.2, R24.1
- net GND_RS485: now also R3.1; no longer R2.1
- net N$1: now also K12.P, K13.P; no longer CH12.P
- net N$10: now also K52.S, K53.S, X4-1.KL; no longer CH61.2, IC1.O8, JP1.13
- net N$11: now also K62.P, K63.P, X4-2.KL; no longer CH51.2, IC1.O7, JP1.11
- net N$12: now also K62.S, K63.S, X4-3.KL; no longer CH41.2, IC1.O6, JP1.9
- net N$13: now also IC2.I1, U1.PA1(ADC1); no longer CH52.P, X3-3.KL
- net N$16: now also IC1.B, R4.2, R6.2; no longer IC2.B, R15.2, R17.2
- net N$18: now also IC2.I2, U1.PA2(ADC2); no longer CH42.P, X3-1.KL
- net N$19: now also IC2.I3, U1.PA3(ADC3); no longer CH62.P, X4-2.KL
- net N$2: now also K12.S, K13.S, X1-2.KL; no longer CH32.S, X2-3.KL
- net N$20: now also IC2.I4, U1.PA4(ADC4); no longer CH62.S, X4-3.KL
- net N$21: now also IC3.I1, U1.PA7/(ADC7/AC0-OUT); no longer JP1.16, U1.PC7(SCK/CLKO/EVO)
- net N$22: now also IC3.I2, U1.PB0(ADC8/AREF); no longer JP1.14, U1.PC6(MISO)
- net N$23: now also IC3.I3, U1.PB1(ADC9); no longer JP1.12, U1.PC5(OC1B/MOSI)
- net N$24: now also IC1.!RE, IC1.DE; no longer IC2.!RE, IC2.DE
- net N$25: now also IC1.D; no longer IC2.D
- net N$26: now also IC1.R; no longer IC2.R
- net N$27: now also IC3.I4, U1.PB2(ADC10); no longer JP1.10, U1.PC4(OC1A/!SS!)
- net N$28: now also JP1.2; no longer JP1.8
- net N$29: now also JP1.1; no longer JP1.6
- net N$3: now also K22.S, K23.S, X2-1.KL; no longer CH22.P, X1-3.KL
- net N$30: now also IC3.I5, U1.PB3(ADC11); no longer JP1.4, U1.PC1(OC0B/XCK0/SCL)
- net N$32: now also IC2.I5, U1.PA5(ADC5); no longer C13.1, C7.+, D5.C, IC3.VI, L1.2
- net N$4: now also K22.P, K23.P, X1-3.KL; no longer CH42.S, X3-2.KL
- net N$5: now also K32.P, K33.P; no longer CH32.P
- net N$6: now also K32.S, K33.S, X2-3.KL; no longer CH52.S, X4-1.KL
- net N$7: now also K42.P, K43.P, X3-1.KL; no longer CH11.2, IC1.O1, JP1.3
- net N$8: now also K42.S, K43.S, X3-2.KL; no longer CH21.2, IC1.O2, JP1.5
- net N$9: now also K52.P, K53.P, X3-3.KL; no longer CH31.2, IC1.O3, JP1.7
- net PROG: no longer C2.1, R32.1
- net RS485_A1: now also IC1.A, R5.2, R8.1; no longer IC2.A, R13.1, R16.2
- net VCC: now also IC2.CD+, IC3.CD+; no longer C4.1, D3.2, D4.A, JP1.1
- net VCC_MAG: now also C4.1, D3.2, D4.A, R2.2; no longer R25.2
- net VCC_MAG_METER: now also R1.2, R2.1, U1.PA0(ADC0/AREF); no longer R24.2, R25.1, U1.PB3(ADC11)
Other:
- note added: "Relay section"
- moved on the sheet: C10, C3, C4, C6, C8, C9, D3, D4, L1, R13, R15, R16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

Commit message: Actor_6_Channel.brd FV
Parts:
- added JP4: (no value), pinhead:PINHD-2X4
- added R21, R22: 0R, rcl:R-EU_R0603
- C3: device rcl:C-EUC0603 -> rcl:C-EUC0603K
Connections:
- net N$24 renamed DE_/RE
- net N$25 renamed TXD
- net N$26 renamed RXD
- net VCC_MAG renamed VCC_BUS
- net VCC_MAG_METER renamed VCC_BUS_METER
- removed net GND_RS485: R3.1, X6.2, X6.6, X6.8, X7.2, X7.6, X7.8
- removed net N$13: IC2.I1, U1.PA1(ADC1)
- removed net N$18: IC2.I2, U1.PA2(ADC2)
- removed net N$19: IC2.I3, U1.PA3(ADC3)
- removed net N$20: IC2.I4, U1.PA4(ADC4)
- removed net N$21: IC3.I1, U1.PA7/(ADC7/AC0-OUT)
- removed net N$22: IC3.I2, U1.PB0(ADC8/AREF)
- removed net N$23: IC3.I3, U1.PB1(ADC9)
- removed net N$27: IC3.I4, U1.PB2(ADC10)
- removed net N$30: IC3.I5, U1.PB3(ADC11)
- removed net N$32: IC2.I5, U1.PA5(ADC5)
- removed net N$33: JP3.3, U1.PDI-CLK/!RESET
- removed net N$34: IC2.I6, U1.PA6(ADC6)
- removed net VCC: IC2.CD+, IC3.CD+
- new net /LA: JP4.1, U1.PD4(!SS!)
- new net CLK: JP4.3, U1.PD7(SCK/CLKO/EVO)
- new net INT: JP4.6, U1.PE2(OC0C)
- new net MOSI: JP4.2, U1.PD5(MOSI)
- new net N$11: JP3.3, U1.PDI-DATA
- new net N$36: C1.2, D1.A, D2.A, IC1.GND, R21.2, R3.2, R6.1
- new net N$37: R22.2, R3.1, X6.2, X6.6, X6.8, X7.2, X7.6, X7.8
- new net PA1: IC3.I6, U1.PA1(ADC1)
- new net PA2: IC3.I5, U1.PA2(ADC2)
- new net PA3: IC3.I4, U1.PA3(ADC3)
- new net PA4: IC3.I3, U1.PA4(ADC4)
- new net PA5: IC3.I2, U1.PA5(ADC5)
- new net PA6: IC3.I1, U1.PA6(ADC6)
- new net PA7: IC2.I6, U1.PA7/(ADC7/AC0-OUT)
- new net PB0: IC2.I5, U1.PB0(ADC8/AREF)
- new net PB1: IC2.I4, U1.PB1(ADC9)
- new net PB2: IC2.I3, U1.PB2(ADC10)
- new net PB3: IC2.I2, U1.PB3(ADC11)
- new net PC0: IC2.I1, U1.PC0(OC0A/SDA)
- new net SCL: JP4.5, U1.PE1(OC0B/SCL)
- new net SDA: JP4.4, U1.PE0(OC0A/SDA)
- net +24V: now also IC2.CD+, IC3.CD+
- net +3V3: now also JP4.7
- net GND: now also JP3.1, JP4.8, R21.1, R22.1; no longer C1.2, D1.A, D2.A, IC1.GND, JP3.4, R3.2, R6.1
- net K1_1: now also IC3.O1; no longer IC2.O2
- net K2_0: now also IC2.O2; no longer IC2.O3
- net K2_1: now also IC3.O2; no longer IC2.O4
- net K3_0: now also IC2.O3; no longer IC2.O5
- net K3_1: now also IC3.O3; no longer IC2.O6
- net K4_0: now also IC2.O4; no longer IC3.O1
- net K4_1: now also IC3.O4; no longer IC3.O2
- net K5_0: now also IC2.O5; no longer IC3.O3
- net K5_1: now also IC3.O5; no longer IC3.O4
- net K6_0: now also IC2.O6; no longer IC3.O5
- net N$14: now also JP3.4, U1.PDI-CLK/!RESET; no longer JP3.1, U1.PDI-DATA
- net PROG: now also U1.PC4(OC1A/!SS!)
Other:
- note added: "TOP PCB SOCKET"
- moved on the sheet: C1, C12, C15, C16, C17, C3, D1, D2, IC1, IC2, IC3, JP2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
